Commit message: Adjust Gazebo sun position for presentation view

File: solar_flower.urdf (robot description, URDF)
Before this commit: robot solar_flower, 6 links, 5 joints
Links:
- added link base_footprint, mass 0.001
- link azimuth_link: mass None -> 0.15
- link base_link: mass None -> 0.25
- link blue_petal_link: mass None -> 0.05
- link green_petal_link: mass None -> 0.05
- link red_petal_link: mass None -> 0.05
- link tilt_link: mass None -> 0.2
Joints:
- added joint base_footprint_to_base_link: type fixed, parent base_footprint, child base_link, origin xyz=0 0 0 rpy=1.5708 0 0
- joint azimuth_joint: origin xyz=0 0.0387 0 rpy=0 0 0 -> xyz=0 0 0 rpy=0 0 0
- joint blue_petal_joint: origin xyz=0 0.2353 0 rpy=0 0 0 -> xyz=-0.0325 0.05995 0 rpy=0 0 0
- joint green_petal_joint: origin xyz=0 0.2463 0 rpy=0 0 0 -> xyz=-0.0325 0.07095 0 rpy=0 0 0
- joint red_petal_joint: origin xyz=0 0.2243 0 rpy=0 0 0 -> xyz=-0.0325 0.04895 0 rpy=0 0 0

File: src/solar_flower_description/urdf/solar_flower.urdf.xacro (robot description, xacro)
@@ -1,7 +1,20 @@
 <?xml version="1.0"?>
 <robot name="solar_flower" xmlns:xacro="http://www.ros.org/wiki/xacro">
-  <!-- Mesh scale: Fusion STL exported in mm, ROS uses meters -->
+<!-- Simple inertial macro for Gazebo spawning -->
+<xacro:macro name="simple_inertial" params="mass ixx iyy izz">
+  <inertial>
+    <origin xyz="0 0 0" rpy="0 0 0"/>
+    <mass value="${mass}"/>
+    <inertia
+      ixx="${ixx}" ixy="0.0" ixz="0.0"
+      iyy="${iyy}" iyz="0.0"
+      izz="${izz}"/>
+  </inertial>
+</xacro:macro>
+<!-- Mesh scale: Fusion STL exported in mm, ROS uses meters -->
   <xacro:property name="mesh_scale" value="0.001 0.001 0.001"/>
-  <link name="base_footprint"/>
+  <link name="base_footprint">
+   <xacro:simple_inertial mass="0.001" ixx="0.000001" iyy="0.000001" izz="0.000001"/>
+  </link>
 <joint name="base_footprint_to_base_link" type="fixed">
   <parent link="base_footprint"/>
@@ -11,4 +24,5 @@
   <!-- Base link -->
   <link name="base_link">
+   <xacro:simple_inertial mass="0.25" ixx="0.0001" iyy="0.0001" izz="0.0001"/>
    <visual>
     <origin xyz="0 0 0" rpy="0 0 0"/>
@@ -23,5 +37,6 @@
   <!-- Azimuth link -->
   <link name="azimuth_link">
-    <visual>
+   <xacro:simple_inertial mass="0.15" ixx="0.00008" iyy="0.00008" izz="0.00008"/>
+   <visual>
       <geometry>
         <mesh filename="package://solar_flower_description/meshes/azimuth_link.stl" scale="${mesh_scale}"/>
@@ -34,4 +49,5 @@
   <!-- Tilt link -->
   <link name="tilt_link">
+   <xacro:simple_inertial mass="0.20" ixx="0.0001" iyy="0.0001" izz="0.0001"/>
    <visual>
     <origin xyz="-0.0325 -0.17535 0" rpy="0 0 0"/>
@@ -46,4 +62,5 @@
   <!-- Red petal -->
   <link name="red_petal_link">
+   <xacro:simple_inertial mass="0.05" ixx="0.00002" iyy="0.00002" izz="0.00002"/>
    <visual>
     <origin xyz="0 -0.2243 0" rpy="0 0 0"/>
@@ -58,4 +75,5 @@
   <!-- Blue petal -->
   <link name="blue_petal_link">
+   <xacro:simple_inertial mass="0.05" ixx="0.00002" iyy="0.00002" izz="0.00002"/>
    <visual>
     <origin xyz="0 -0.2353 0" rpy="0 0 0"/>
@@ -70,4 +88,5 @@
   <!-- Green petal -->
   <link name="green_petal_link">
+   <xacro:simple_inertial mass="0.05" ixx="0.00002" iyy="0.00002" izz="0.00002"/>
    <visual>
     <origin xyz="0 -0.2463 0" rpy="0 0 0"/>
